File: hw/rev2/pcb/TrueStrike56/TrueStrike56.kicad_pcb (KiCad board)
At the start: 2 copper layers, 258 x 110.9 mm, 133 parts, among them SW1 SW_Push, SW2 RotaryEncoder_Switch, U1 ProMicro, U10 4053, U11 ER_OLEDM0.91_1x-I2C, U2 74HC4051, U3 74HC4051, U4 74HC4051, U5 74HC4051, U6 74HC4051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

Commit message: Add mounting holes to PCB
Parts:
- added H1: MountingHole, MountingHole:MountingHole_3.5mm, F.Cu at (95.1, 73.2)
- added H2: MountingHole, MountingHole:MountingHole_3.5mm, F.Cu at (170.9, 80.5)
- added H3: MountingHole, MountingHole:MountingHole_3.5mm, F.Cu at (93.9, 134.1)
- added H4: MountingHole, MountingHole:MountingHole_3.5mm, F.Cu at (171.7, 140.1)
- added H5: MountingHole, MountingHole:MountingHole_3.5mm, F.Cu at (229.1, 80.7)
- added H6: MountingHole, MountingHole:MountingHole_3.5mm, F.Cu at (304.9, 73.4)
- added H7: MountingHole, MountingHole:MountingHole_3.5mm, F.Cu at (228.1, 140.2)
- added H8: MountingHole, MountingHole:MountingHole_3.5mm, F.Cu at (305.8, 134.6)
