File: hw/rev2/pcb/TrueStrike56/TrueStrike56.kicad_sch (KiCad schematic)
At the start: 132 parts, among them SW1 SW_Push, SW2 RotaryEncoder_Switch, U1 ProMicro, U10 4053, U11 ER_OLEDM0.91_1x-I2C, U2 74HC4051, U3 74HC4051, U4 74HC4051, U5 74HC4051, U6 74HC4051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

Commit message: Add mounting holes to PCB
Parts:
- added H1, H2, H3, H4, H5, H6, H7, H8: MountingHole, MountingHole:MountingHole_3.5mm, symbol Mechanical:MountingHole
